Commit message: viconball mass fix.

File: vicon/matlab-model/ball.urdf (robot description, URDF)
Before this commit: robot viconBall, 1 links, 0 joints
Links:
- removed link Body
- added link Ball, mass 3; collision sphere radius=0.0001; visual sphere radius=0.1

Commit message: Visualization with right trajs

File: vicon/matlab-model/ball.urdf (robot description, URDF)
Before this commit: robot viconBall, 1 links, 0 joints
Links:
- link Ball: geometry collision sphere radius=0.0001; visual sphere radius=0.067

Commit message: HuboControllerGain

File: vicon/matlab-model/ball.urdf (robot description, URDF)
Before this commit: robot viconBall, 1 links, 0 joints
Links:
- link Ball: geometry collision sphere radius=0.0001; visual sphere radius=0.04

Commit message: Tuned trajectory matching

File: vicon/matlab-model/ball.urdf (robot description, URDF)
Before this commit: robot viconBall, 1 links, 0 joints
Links:
- link Ball: mass 1 -> 0.1; geometry collision sphere radius=0.04; visual sphere radius=0.04
